File: board/music_player.kicad_sch (KiCad schematic)
At the start: 28 parts, among them J1 Micro_SD_Card_Det1, J2 USB_C_Receptacle_PowerOnly_6P, SW1 SW_SPDT, U1 STM32F401RET6, U2 PCM5102A, Y1 8MHz

Commit message: added kicad schematic
Parts:
- added R5: 47k, symbol Device:R
Connections:
- net +3.3V: now also R5.1
- net SD_SCK: now also R5.2
Other:
- moved on the sheet: C13, C14, J1, J2, R2, R3, R4, R6, R7, R8, U2
